File: Micr0.kicad_pcb (KiCad board)
At the start: 2 copper layers, 33.6 x 50 mm, 56 parts, among them J1 AudioJack2, J2 AudioJack2, J3 Barrel_Jack_Switch, Q1 BC807, Q2 MMBF170, SW1 SW_DPDT_x2, U1 TL074, U2 LM13700

Commit message: Added gerbers
Routing:
- net Net-(U1A-+): track 24.3 -> 23.6 mm
- net +9V: track 85.6 -> 86.3 mm
Other:
- outline, holes or cut-outs redrawn
- board text added: "JLCJLCJLCJLC"
- board text added: "https://github.com/ Secret624/Micr0"
